Commit message: added trees to specified polygons

File: generation/Terrain_Generation/terrain_features/lowpoly_tree.urdf (robot description, URDF)
Before this commit: robot low_poly_tree, 1 links, 0 joints
Links:
- removed link low_poly_tree_link
- added link base, mass 1000.0; collision mesh filename=tree_trunk.obj scale=1 1 1; visual mesh filename=tree_trunk.obj scale=1 1 1
- added link canopy_link, mass 500.0; visual mesh filename=tree_canopy.obj scale=2 2 2
Joints:
- added joint trunk_to_canopy: type fixed, parent base, child canopy_link, origin xyz=0 0 10.0 rpy=0 0 0

Commit message: Adding features to the scene

File: generation/Terrain_Generation/terrain_features/lowpoly_tree.urdf (robot description, URDF)
Before this commit: robot low_poly_tree, 2 links, 1 joints
Links:
- removed link base
- removed link canopy_link
- added link canopy, mass 5.0; collision mesh filename=tree_canopy.obj scale=1 1 1; visual mesh filename=tree_canopy.obj scale=1 1 1
- added link trunk, mass 5.0; collision mesh filename=tree_trunk.obj scale=1 1 1; visual mesh filename=tree_trunk.obj scale=1 1 1
Joints:
- joint trunk_to_canopy: child canopy_link -> canopy; origin xyz=0 0 10.0 rpy=0 0 0 -> xyz=0 0 5.0 rpy=0 0 0; parent base -> trunk
